Commit message: Odom II

File: ros2_ws/src/mecanum4_description/urdf/mecanum4_lidar.urdf (robot description, URDF)
Before this commit: robot mecanum4_lidar, 7 links, 6 joints
Joints:
- joint wheel_fl_joint: type continuous -> fixed
- joint wheel_fr_joint: type continuous -> fixed
- joint wheel_rl_joint: type continuous -> fixed
- joint wheel_rr_joint: type continuous -> fixed

Commit message: update URDF to SIM

File: ros2_ws/src/mecanum4_description/urdf/mecanum4_lidar.urdf (robot description, URDF)
Before this commit: robot mecanum4_lidar, 7 links, 6 joints
Links:
- link wheel_fl_link: mass None -> 0.5; geometry collision cylinder length=0.03 radius=0.05; visual cylinder length=0.03 radius=0.05
- link wheel_fr_link: mass None -> 0.5; geometry collision cylinder length=0.03 radius=0.05; visual cylinder length=0.03 radius=0.05
- link wheel_rl_link: mass None -> 0.5; geometry collision cylinder length=0.03 radius=0.05; visual cylinder length=0.03 radius=0.05
- link wheel_rr_link: mass None -> 0.5; geometry collision cylinder length=0.03 radius=0.05; visual cylinder length=0.03 radius=0.05
Joints:
- joint wheel_fl_joint: type fixed -> continuous
- joint wheel_fr_joint: type fixed -> continuous
- joint wheel_rl_joint: type fixed -> continuous
- joint wheel_rr_joint: type fixed -> continuous

Commit message: ros2 control can run

File: ros2_ws/src/mecanum4_description/urdf/mecanum4_lidar.urdf (robot description, URDF)
Before this commit: robot mecanum4_lidar, 7 links, 6 joints
Links:
- link base_link: mass None -> 0.001
- link laser_frame: mass None -> 0.10; geometry collision cylinder length=0.05 radius=0.035; visual cylinder length=0.05 radius=0.035

Commit message: change urdf and control it

File: ros2_ws/src/mecanum4_description/urdf/mecanum4_lidar.urdf (robot description, URDF)
Before this commit: robot mecanum4_lidar, 7 links, 6 joints
Joints:
- joint wheel_fl_joint: origin xyz=0.16 0.13 0.05 rpy=0 0 0 -> xyz=0.16 0.18 0.05 rpy=0 0 0
- joint wheel_fr_joint: origin xyz=0.16 -0.13 0.05 rpy=0 0 0 -> xyz=0.16 -0.18 0.05 rpy=0 0 0
- joint wheel_rl_joint: origin xyz=-0.16 0.13 0.05 rpy=0 0 0 -> xyz=-0.16 0.18 0.05 rpy=0 0 0
- joint wheel_rr_joint: origin xyz=-0.16 -0.13 0.05 rpy=0 0 0 -> xyz=-0.16 -0.18 0.05 rpy=0 0 0

Commit message: can walk

File: ros2_ws/src/mecanum4_description/urdf/mecanum4_lidar.urdf (robot description, URDF)
Before this commit: robot mecanum4_lidar, 7 links, 6 joints
Links:
- removed link chassis_link
- link base_link: mass 0.001 -> 5.0; geometry collision box size=0.40 0.30 0.12; visual box size=0.40 0.30 0.12
- link wheel_fl_link: geometry collision sphere radius=0.05; visual cylinder length=0.03 radius=0.05
- link wheel_fr_link: geometry collision sphere radius=0.05; visual cylinder length=0.03 radius=0.05
- link wheel_rl_link: geometry collision sphere radius=0.05; visual cylinder length=0.03 radius=0.05
- link wheel_rr_link: geometry collision sphere radius=0.05; visual cylinder length=0.03 radius=0.05
Joints:
- removed joint base_to_chassis
- joint wheel_fl_joint: parent chassis_link -> base_link
- joint wheel_fr_joint: parent chassis_link -> base_link
- joint wheel_rl_joint: parent chassis_link -> base_link
- joint wheel_rr_joint: parent chassis_link -> base_link

Commit message: side walk

File: ros2_ws/src/mecanum4_description/urdf/mecanum4_lidar.urdf (robot description, URDF)
Before this commit: robot mecanum4_lidar, 6 links, 5 joints
Links:
- link wheel_fl_link: geometry collision cylinder length=0.03 radius=0.05; visual cylinder length=0.03 radius=0.05
- link wheel_fr_link: geometry collision cylinder length=0.03 radius=0.05; visual cylinder length=0.03 radius=0.05
- link wheel_rl_link: geometry collision cylinder length=0.03 radius=0.05; visual cylinder length=0.03 radius=0.05
- link wheel_rr_link: geometry collision cylinder length=0.03 radius=0.05; visual cylinder length=0.03 radius=0.05

Commit message: dock spear {

File: ros2_ws/src/mecanum4_description/urdf/mecanum4_lidar.urdf (robot description, URDF)
Before this commit: robot mecanum4_lidar, 8 links, 7 joints
Joints:
- joint camera_joint: origin xyz=0.21 0 0.15 rpy=0 0 0 -> xyz=0.21 0 0.25 rpy=0 0 0
- joint laser_joint: origin xyz=0.10 0.00 0.20 rpy=0 0 0 -> xyz=0.10 0.00 0.10 rpy=0 0 0

Commit message: decistion yolo

File: ros2_ws/src/mecanum4_description/urdf/mecanum4_lidar.urdf (robot description, URDF)
Before this commit: robot mecanum4_lidar, 8 links, 7 joints
Joints:
- joint laser_joint: origin xyz=0.10 0.00 0.10 rpy=0 0 0 -> xyz=0.00 0.00 0.10 rpy=0 0 0
